Commit message: fix: fixes name of hip joint

File: bolt_description/urdf/body.xacro (robot description, xacro)
@@ -1,11 +1,11 @@
 <?xml version="1.0"?>
 <robot xmlns:xacro="http://playerstage.sourceforge.net/gazebo/xmlschema/#interface" name="bolt">
-  <joint name="base_joint" type="fixed">
-    <parent link="base_link"/>
-    <child link="body"/>
-    <origin rpy="0 0 0" xyz="0 0 0"/>
-    <axis xyz="0 0 1"/>
-  </joint>
   <xacro:macro name="body">
+    <joint name="base_joint" type="fixed">
+      <parent link="base_link"/>
+      <child link="body"/>
+      <origin rpy="0 0 0" xyz="0 0 0"/>
+      <axis xyz="0 0 1"/>
+    </joint>
     <link name="body">
       <inertial>

File: bolt_description/urdf/bolt.urdf.xacro (robot description, xacro)
@@ -34,9 +34,9 @@
   <ros2_control name="bolt_mujoco_simulation" type="system">
     <xacro:joint_interface name="FR_HAA" p="500" d="0.1" />
-    <xacro:joint_interface name="FR_HFA" p="1" d="0.1" />
+    <xacro:joint_interface name="FR_HFE" p="1" d="0.1" />
     <xacro:joint_interface name="FR_KFE" p="1" d="0.1" />
     <!-- <xacro:joint_interface name="FR_ANKLE" p="10" d="0.1" /> -->
     <xacro:joint_interface name="FL_HAA" p="500" d="0.1" />
-    <xacro:joint_interface name="FL_HFA" p="1" d="0.1" />
+    <xacro:joint_interface name="FL_HFE" p="1" d="0.1" />
     <xacro:joint_interface name="FL_KFE" p="1" d="0.1" />
     <!-- <xacro:joint_interface name="FL_ANKLE" p="10" d="0.1" /> -->
