Commit message: premature commit

File: bolt_description/urdf/bolt.urdf.xacro (robot description, xacro)
@@ -1,2 +1,3 @@
+<?xml version="1.0"?>
 <robot name="bolt" xmlns:xacro="http://playerstage.sourceforge.net/gazebo/xmlschema/#interface">
   <xacro:property name="color_name" value="grey" />
@@ -6,62 +7,46 @@
   <xacro:property name="has_passive_ankle" value="false" />
   <link name="base_link"/>
-  <joint name="base_joint" type="fixed">
-    <parent link="base_link"/>
-    <child link="body"/>
-    <origin rpy="0 0 0" xyz="0 0 0"/>
-    <axis xyz="0 0 1"/>
-  </joint>
-  <link name="body">
-      <inertial>
-          <origin xyz="0 0 0" rpy="0 0 0" />
-          <mass value="0.61436936"/>
-          <inertia ixx="0.00578574" ixy="0.0" ixz="0.0"
-                                    iyy="0.01938108" iyz="0.0"
-                                                    izz="0.02476124"
-          />
-      </inertial>
-      <visual name="body_visual">
-          <origin xyz="0 0 0" rpy="0 0 0" />
-          <geometry>
-            <mesh filename="package://bolt_description/meshes/bolt_body.stl"/>
-          </geometry>
-          <material name="${color_name}">
-              <color rgba="${color} ${opacity}"/>
-          </material>
-      </visual>
-      <collision name="body_collision">
-          <origin xyz="0 0 0" rpy="0 0 0" />
-          <geometry>
-            <mesh filename="package://bolt_description/meshes/bolt_body.stl"/>
-          </geometry>
-          <material name="${color_name}">
-              <color rgba="${color} ${opacity}"/>
-          </material>
-      </collision>
-  </link>
+  <xacro:include filename="body.xacro"/>
   <xacro:include filename="leg.xacro"/>
+  <xacro:body />
   <xacro:leg
-      prefix="FL"
-      is_front="true"
-      is_right="false"
-      has_side_motion="true"
-      color_name="${color_name}"
-      color="${color}"
-      opacity="${opacity}"
-      new_leg="${new_leg}"
-      has_passive_ankle="${has_passive_ankle}"/>
+    prefix="FL"
+    is_front="true"
+    is_right="false"
+    has_side_motion="true"
+    color_name="${color_name}"
+    color="${color}"
+    opacity="${opacity}"
+    new_leg="${new_leg}"
+    has_passive_ankle="${has_passive_ankle}"/>
   <xacro:leg
-      prefix="FR"
-      is_front="true"
-      is_right="true"
-      has_side_motion="true"
-      color_name="${color_name}"
-      color="${color}"
-      opacity="${opacity}"
-      new_leg="${new_leg}"
-      has_passive_ankle="${has_passive_ankle}"/>
+    prefix="FR"
+    is_front="true"
+    is_right="true"
+    has_side_motion="true"
+    color_name="${color_name}"
+    color="${color}"
+    opacity="${opacity}"
+    new_leg="${new_leg}"
+    has_passive_ankle="${has_passive_ankle}"/>
+  <xacro:include filename="$(find bolt_description)/urdf/joint.xacro"/>
+  <ros2_control name="bolt_mujoco_simulation" type="system">
+    <xacro:joint_interface name="FR_HAA" p="1000" d="0.5" />
+    <xacro:joint_interface name="FR_HFA" p="1000" d="0.5" />
+    <xacro:joint_interface name="FR_KFE" p="1000" d="0.5" />
+    <!-- <xacro:joint_interface name="FR_ANKLE" p="1000" d="0.5" /> -->
+    <xacro:joint_interface name="FL_HAA" p="1000" d="0.5" />
+    <xacro:joint_interface name="FL_HFA" p="1000" d="0.5" />
+    <xacro:joint_interface name="FL_KFE" p="1000" d="0.5" />
+    <!-- <xacro:joint_interface name="FL_ANKLE" p="1000" d="0.5" /> -->
+    <hardware>
+      <plugin>bolt_mujoco_simulation/Simulator</plugin>
+      <!-- <param name="mujoco_model">$(arg mujoco_model)</param> -->
+      <param name="mujoco_model">/home/ws/src/bolt_ros2/bolt_mujoco_simulation/etc/world.xml</param>
+    </hardware>
+  </ros2_control>
   <mujoco>
-      <!-- TODO: fix this path -->
-      <compiler
+    <!-- TODO: fix this path -->
+    <compiler
       meshdir="/home/ws/src/bolt_description/resource/meshes"
       discardvisual="false" />

File: bolt_description/urdf/leg.xacro (robot description, xacro)
@@ -380,57 +380,4 @@
     </link>
     <!-- END FOOT LINK -->
-    <ros2_control name="bolt" type="system">
-      <hardware>
-        <plugin>
-          <!-- {Name_Space}/{Class_Name}-->
-        </plugin>
-      </hardware>
-      <joint name="${prefix}_HAA">
-        <command_interface name="position">
-          <param name="min">{-0.5*pi}</param>
-          <param name="max">{0.5*pi}</param>
-        </command_interface>
-        <!-- additional command interfaces ... -->
-        <state_interface name="position">
-          <param name="initial_value">0.0</param>
-        </state_interface>
-        <!-- additional state interfaces ... -->
-      </joint>
-      <joint name="${prefix}_HFA">
-        <command_interface name="position">
-          <param name="min">{-0.5*pi}</param>
-          <param name="max">{0.5*pi}</param>
-        </command_interface>
-        <!-- additional command interfaces ... -->
-        <state_interface name="position">
-          <param name="initial_value">0.0</param>
-        </state_interface>
-        <!-- additional state interfaces ... -->
-      </joint>
-      <joint name="${prefix}_KFE">
-        <command_interface name="position">
-          <param name="min">{-1*pi}</param>
-          <param name="max">{1*pi}</param>
-        </command_interface>
-        <!-- additional command interfaces ... -->
-        <state_interface name="position">
-          <param name="initial_value">0.0</param>
-        </state_interface>
-        <!-- additional state interfaces ... -->
-      </joint>
-      <joint name="${prefix}_ANKLE">
-        <command_interface name="position">
-          <param name="min">{-0.5*pi}</param>
-          <param name="max">{0.5*pi}</param>
-        </command_interface>
-        <!-- additional command interfaces ... -->
-        <state_interface name="position">
-          <param name="initial_value">0.0</param>
-        </state_interface>
-        <!-- additional state interfaces ... -->
-      </joint>
-      <!-- additional joints ...-->
-      <!-- additional hardware/sensors ...-->
-    </ros2_control>
   </xacro:macro>
 </robot>

Commit message: removes dampening and stiffness values

File: bolt_description/urdf/bolt.urdf.xacro (robot description, xacro)
@@ -32,12 +32,12 @@
   <xacro:include filename="$(find bolt_description)/urdf/joint.xacro"/>
   <ros2_control name="bolt_mujoco_simulation" type="system">
-    <xacro:joint_interface name="FR_HAA" p="1000" d="0.5" />
-    <xacro:joint_interface name="FR_HFA" p="1000" d="0.5" />
-    <xacro:joint_interface name="FR_KFE" p="1000" d="0.5" />
-    <!-- <xacro:joint_interface name="FR_ANKLE" p="1000" d="0.5" /> -->
-    <xacro:joint_interface name="FL_HAA" p="1000" d="0.5" />
-    <xacro:joint_interface name="FL_HFA" p="1000" d="0.5" />
-    <xacro:joint_interface name="FL_KFE" p="1000" d="0.5" />
-    <!-- <xacro:joint_interface name="FL_ANKLE" p="1000" d="0.5" /> -->
+    <xacro:joint_interface name="FR_HAA" />
+    <xacro:joint_interface name="FR_HFA" />
+    <xacro:joint_interface name="FR_KFE" />
+    <!-- <xacro:joint_interface name="FR_ANKLE" /> -->
+    <xacro:joint_interface name="FL_HAA" />
+    <xacro:joint_interface name="FL_HFA" />
+    <xacro:joint_interface name="FL_KFE" />
+    <!-- <xacro:joint_interface name="FL_ANKLE" /> -->
     <hardware>
       <plugin>bolt_mujoco_simulation/Simulator</plugin>

File: bolt_description/urdf/joint.xacro (robot description, xacro)
@@ -1,5 +1,5 @@
 <?xml version="1.0"?>
 <robot xmlns:xacro="http://www.ros.org/wiki/xacro">
-  <xacro:macro name="joint_interface" params="name p d">
+  <xacro:macro name="joint_interface" params="name">
     <joint name="${name}">
       <command_interface name="position">
@@ -11,6 +11,4 @@
         <param name="max">1</param>
       </command_interface>
-      <param name="p">${p}</param>
-      <param name="d">${d}</param>
       <state_interface name="position"/>
       <state_interface name="velocity"/>

Commit message: restores stiffening and dampening parameters

File: bolt_description/urdf/bolt.urdf.xacro (robot description, xacro)
@@ -32,12 +32,12 @@
   <xacro:include filename="$(find bolt_description)/urdf/joint.xacro"/>
   <ros2_control name="bolt_mujoco_simulation" type="system">
-    <xacro:joint_interface name="FR_HAA" />
-    <xacro:joint_interface name="FR_HFA" />
-    <xacro:joint_interface name="FR_KFE" />
-    <!-- <xacro:joint_interface name="FR_ANKLE" /> -->
-    <xacro:joint_interface name="FL_HAA" />
-    <xacro:joint_interface name="FL_HFA" />
-    <xacro:joint_interface name="FL_KFE" />
-    <!-- <xacro:joint_interface name="FL_ANKLE" /> -->
+    <xacro:joint_interface name="FR_HAA" p="10" d="0.1" />
+    <xacro:joint_interface name="FR_HFA" p="10" d="0.1" />
+    <xacro:joint_interface name="FR_KFE" p="10" d="0.1" />
+    <!-- <xacro:joint_interface name="FR_ANKLE" p="10" d="0.1" /> -->
+    <xacro:joint_interface name="FL_HAA" p="10" d="0.1" />
+    <xacro:joint_interface name="FL_HFA" p="10" d="0.1" />
+    <xacro:joint_interface name="FL_KFE" p="10" d="0.1" />
+    <!-- <xacro:joint_interface name="FL_ANKLE" p="10" d="0.1" /> -->
     <hardware>
       <plugin>bolt_mujoco_simulation/Simulator</plugin>

File: bolt_description/urdf/joint.xacro (robot description, xacro)
@@ -1,5 +1,5 @@
 <?xml version="1.0"?>
 <robot xmlns:xacro="http://www.ros.org/wiki/xacro">
-  <xacro:macro name="joint_interface" params="name">
+  <xacro:macro name="joint_interface" params="name p d">
     <joint name="${name}">
       <command_interface name="position">
@@ -11,4 +11,6 @@
         <param name="max">1</param>
       </command_interface>
+      <param name="p">${p}</param>
+      <param name="d">${d}</param>
       <state_interface name="position"/>
       <state_interface name="velocity"/>

Commit message: feat: implements PD+ control for simulation

File: bolt_description/urdf/bolt.urdf.xacro (robot description, xacro)
@@ -33,11 +33,11 @@
   <xacro:include filename="$(find bolt_description)/urdf/joint.xacro"/>
   <ros2_control name="bolt_mujoco_simulation" type="system">
-    <xacro:joint_interface name="FR_HAA" p="1" d="0.1" />
-    <xacro:joint_interface name="FR_HFE" p="1" d="0.1" />
-    <xacro:joint_interface name="FR_KFE" p="1" d="0.1" />
+    <xacro:joint_interface name="FR_HAA" p="1" d="0.1" t="0.05"/>
+    <xacro:joint_interface name="FR_HFE" p="1" d="0.1" t="0.05"/>
+    <xacro:joint_interface name="FR_KFE" p="1" d="0.1" t="0.05"/>
     <!-- <xacro:joint_interface name="FR_ANKLE" p="10" d="0.1" /> -->
-    <xacro:joint_interface name="FL_HAA" p="1" d="0.1" />
-    <xacro:joint_interface name="FL_HFE" p="1" d="0.1" />
-    <xacro:joint_interface name="FL_KFE" p="1" d="0.1" />
+    <xacro:joint_interface name="FL_HAA" p="1" d="0.1" t="0.05"/>
+    <xacro:joint_interface name="FL_HFE" p="1" d="0.1" t="0.05"/>
+    <xacro:joint_interface name="FL_KFE" p="1" d="0.1" t="0.05"/>
     <!-- <xacro:joint_interface name="FL_ANKLE" p="10" d="0.1" /> -->
     <xacro:if value="$(arg sim)">

File: bolt_description/urdf/joint.xacro (robot description, xacro)
@@ -1,5 +1,5 @@
 <?xml version="1.0"?>
 <robot xmlns:xacro="http://www.ros.org/wiki/xacro">
-  <xacro:macro name="joint_interface" params="name p d">
+  <xacro:macro name="joint_interface" params="name p d t">
     <joint name="${name}">
       <command_interface name="position">
@@ -11,6 +11,11 @@
         <param name="max">1</param>
       </command_interface>
+      <command_interface name="effort">
+        <param name="min">-100</param>
+        <param name="max">100</param>
+      </command_interface>
       <param name="p">${p}</param>
       <param name="d">${d}</param>
+      <param name="t">${d}</param>
       <state_interface name="position"/>
       <state_interface name="velocity"/>

Commit message: refactor: more accurately specifies prior sensor_link frames as imu_link

File: bolt_description/urdf/bolt.urdf.xacro (robot description, xacro)
@@ -12,5 +12,6 @@
   <xacro:include filename="sensor.xacro"/>
   <xacro:body />
-  <xacro:sensor />
+  <xacro:sensor
+    link_name="imu_link"/>
   <xacro:leg
     prefix="FL"

File: bolt_description/urdf/sensor.xacro (robot description, xacro)
@@ -1,12 +1,12 @@
 <?xml version="1.0"?>
 <robot xmlns:xacro="http://playerstage.sourceforge.net/gazebo/xmlschema/#interface" name="bolt">
-  <xacro:macro name="sensor">
-    <joint name="sensor_joint" type="fixed">
+  <xacro:macro name="sensor" params="link_name">
+    <joint name="${link_name}_joint" type="fixed">
       <parent link="base_link"/>
-      <child link="sensor_link"/>
+      <child link="${link_name}"/>
       <origin rpy="0 0 0" xyz="0 0 0"/>
       <axis xyz="0 0 1"/>
     </joint>
-    <link name="sensor_link">
+    <link name="${link_name}">
       <inertial>
         <origin xyz="0 0 0" rpy="0 0 0" />
